File: MilliToney.sch (EAGLE design)
At the start: 72 parts, among them J1 BANANA_CONN, J2 BANANA_CONN, J3 BANANA_CONN, J4 BANANA_CONN, J5 BANANA_CONN, J6 BANANA_CONN, J7 BANANA_CONN, J8 BANANA_CONN, Q1 BC807-16LT1SMD, U1 OPA335AIDBVT, U2 TLV431BIDBZR

Commit message: Committing latest updates
Committing latest updates. dual footprints buzzer and battery, updated
other parts. added 5x5 footprint for board
Parts:
- removed D7: 2.7V, SparkFun-DiscreteSemi:DIODE-ZENER3.3V
- removed D8: 0.5A SOD323F, adafruit:DIODESOD-323F
- removed J4, J5, J6, J7, J8: BANANA_CONN, SparkFun-Connectors:BANANA_CONN
- removed PAD1, PAD2, PAD3, PAD4: MOUNT_HOLE, wirepad:3,81/1,4
- removed TP7, TP8, TP9: TP_1MM_TH", TP_1MM_TH:TP_1MM_TH"
- added BAT1: CR2032, SparkFun-Electromechanical:BATTERYFOB
- added BAT2: CR2032, kzh20_lithium_batterie_holder:2032
- added C11: 10nF, rcl:C-EUC0402K
- added C12: 10uF, rcl:C-EUC0603
- added C13: 100nF, rcl:C-EUC0402K
- added C14: 10uF, rcl:C-EUC0603K
- added PCB1: PCB_DP_SQUARE-5X5, dp_devices:PCB_DP_SQUARE-5X5
- added R21: 1k, rcl:R-EU_R0402
- added SP4: KSS1201, buzzer:KSS1201
- added U$3, U$4: FIDUCIAL, adafruit:FIDUCIAL
- added U3: OPA335AIDBVT, Texas Instruments_By_element14_Batch_1:OPA335AIDBVT
- added U5: Comparator, MCP6541_SOT23-5:MCP6541T-I/OT
- added VR1: (no value), bourns:3386-F
- added VR3: 1k, bourns:3386-F
- C1: value 100n -> DNF
- C10: value 100n -> 100nF
- C2: value 10n -> 10uF; device rcl:C-EUC0402K -> rcl:C-EUC0603
- C4: value 100p -> 470pF
- C5: value (none) -> 100n
- C6: value (none) -> 10n
- C7: value (none) -> 100p; device rcl:C-EUC0603K -> rcl:C-EUC0402K
- C9: value 100n -> 10n
- D1: value 1N4148W_SOD123 -> 0.5A SOD323F; device adafruit:DIODE_SOD-123FL -> adafruit:DIODESOD-323F; MF (none) -> NXP; MPN (none) -> PMEG3010EJ,115; OC_FARNELL (none) -> 1757770
- D2, D5: value 2.7V -> 1N4148W_SOD123; device SparkFun-DiscreteSemi:DIODE-ZENER3.3V -> adafruit:DIODE_SOD-123FL
- J3: value BANANA_CONN -> BNCPTH; device SparkFun-Connectors:BANANA_CONN -> SparkFun-Connectors:BNCPTH; OC_FARNELL unknown -> (none)
- LED1: value GREEN_LED -> (none); device P-LCC-2_Shorter:LEDP-LCC-2 -> led:LEDSML0603; MF OSRAM -> (none); MPN LGT67K-H2K1-24-Z -> (none); OC_FARNELL 1226376 -> (none)
- R12: value NOFIT -> (none)
- R13: value (none) -> 2k
- R15, R4: value (none) -> 1M
- R16: value (none) -> 47k
- R17: value (none) -> 100k
- R18: value (none) -> 1k
- R19: value (none) -> 330R; device bourns:3386-F -> rcl:R-EU_R0402
- R2: value (none) -> 2k; device bourns:3386-F -> rcl:R-EU_R0402
- R20: value 2k -> 47k
- R8: device rcl:R-EU_R0402 -> rcl:R-EU_R0603
- SG1: value BUZZERSMD3 -> BUZZERBUZZER-KMTG1203; device SparkFun-Electromechanical:BUZZERSMD3 -> KMTG1203:BUZZERBUZZER-KMTG1203
- TP1, TP3: MF MULTICOMP -> (none); MPN TEST-3 -> (none); OC_FARNELL 1702006 -> (none)
- U$1: value MCP6001T-E/OT -> FIDUCIAL; device Microchip_By_element14_Batch_1:MCP6001T-E/OT -> adafruit:FIDUCIAL
- U$2: value 2032 -> FIDUCIAL; device kzh20_lithium_batterie_holder:2032 -> adafruit:FIDUCIAL; MF RENATA -> (none); MPN SMTU 2032-LF -> (none); OC_FARNELL 1216354 -> (none)
- U1: value OPA335AIDBVT -> NCP303LSN09; device Texas Instruments_By_element14_Batch_1:OPA335AIDBVT -> SparkFun-DigitalIC:NCP303LSN09
- U4: value (none) -> MCP6001T-E/OT; device MCP6541_SOT23-5:MCP6541T-I/OT -> Microchip_By_element14_Batch_1:MCP6001T-E/OT
Connections:
- removed net +2.5V_REF: J3.1, TP1.1
- removed net HI_OUT: J8.1, R9.1, TP4.1
- removed net HI_SENSE: C5.1, J1.1, R7.1, TP5.1
- removed net N$10: C4.2, D7.A, R5.1, R6.2, U1.OUT
- removed net N$12: R15.1, R16.1, R18.2, R19.2, TP8.1, U4.OUT
- removed net N$13: D5.A, R13.1, R20.1, R4.2, U$1.VOUT
- new net N$24: C11.2, Q1.C, R15.1, R19.2, TP6.1, U5.VIN+
- new net N$27: R8.2, TP1.1
- new net N$30: LED2.A, R2.1
- new net VIN: C4.1, J2.1, R3.1, R4.2, R5.1
- new net VOUTA: C7.2, R10.1, R9.2, U3.OUT
- new net VOUTB: C9.1, D4.C, J3.OUT, R10.2, U4.VIN+
- new net VOUT_COMP: D5.C, R20.1, R21.2, U5.OUT, VR3.1, VR3.2
- new net VOUT_DRIVE: R12.2, R13.1, R14.1, U4.VOUT
- new net VREF: C8.1, D6.C, R3.2, R7.1, U2.CATHODE, U2.REF
- net GND: now also BAT1.-, BAT2.-, C11.1, C13.1, C3.1, C4.2, C5.1, C8.2, C9.2, D1.A, D4.A, D6.A, J1.1, J3.GND, LED2.C, R15.2, R16.2, R4.1, R6.1, SP4.2, U1.GND, U3.V-, U5.VSS; no longer C5.2, C6.1, C8.1, C9.1, D2.A, D8.A, J2.1, J5.1, J6.1, J7.1, LED1.C, PAD1.P, PAD2.P, PAD3.P, PAD4.P, R12.2, R17.2, R8.1, TP3.1, TP6.1, TP7.1, U$1.VSS, U$2.-, U1.V-
- net N$1: now also BAT1.+, BAT2.+, F1.1; no longer S1.P, U$2.+
- net N$11: now also R12.1, VR1.3; no longer R2.2, R4.1
- net N$14: now also U4.VIN-, VR1.1, VR1.2; no longer D4.A, R2.1, U$1.VIN-
- net N$16: now also LED1.C, U1.RST; no longer D4.C, D5.C
- net N$17: now also C12.2, R14.2, R17.2, TP5.1; no longer R13.2, R3.2
- net N$18: now also R18.1; no longer R14.1
- net N$19: now also D1.C, F1.2, S1.P; no longer C6.2, Q1.C, R15.2
- net N$20: now also C1.1, U1.CD; no longer D6.C, D7.C
- net N$21: now also R16.1, R20.2, U5.VIN-; no longer R16.2, R17.1
- net N$22: now also C14.1, VR3.3; no longer C7.1, R19.3, TP9.1
- net N$23: now also R13.2; no longer R20.2
- net N$3: now also C14.2, SP4.1; no longer C7.2
- net N$5: now also R8.1, TP3.1; no longer F1.1, S1.S
- net N$6: now also C6.2, D2.A, D3.C, R5.2, U3.+IN; no longer C3.2, D1.C, D3.A, R12.1, R7.2, U1.+IN
- net N$7: now also TP2.1, TP4.1; no longer C1.1, R10.1, R9.2, U2.CATHODE, U2.REF
- net N$8: now also D5.A, R19.1; no longer C2.1, D2.C, J4.1, R5.2, TP2.1, U$1.VIN+
- net N$9: now also C6.1, C7.1, D2.C, D3.A, R6.2, R9.1, U3.-IN; no longer C3.1, C4.1, D1.A, D3.C, D6.A, R6.1, R8.2, U1.-IN
- net VCC: now also C12.1, C13.2, C2.1, C3.2, C5.2, R17.1, R18.2, R2.2, R21.1, R7.2, S1.S, U1.IN, U3.V+, U5.VDD; no longer C8.2, C9.2, D8.C, F1.2, R10.2, R14.2, R18.1, R3.1, U$1.VDD, U1.V+
Other:
- note added: "BD4827G-TR"
- note added: "CHECK THE FOLLOWING footprints:- Switch = Fully Checked, Diode = checked Fuse = checked Battery con = checked"
- note added: "DETERMINE IF THE COMPARATOR CAN SINK ENOUGH CURRENT DETERMINE IF A TRANSISTOR IS NEEDED ON THE OUTPUT, DETERMINE IF AC COUPLING WILL REDUCE DC CURRENT DRAW"
- note added: "DUAL FOOTPRINT. ONLY FIT ONE BATTERY HOLDER."
- note added: "FIDUCIALS"
- note added: "FIT EITHER Q1 OR R21"
- note added: "SICK OF BEIGE DP5050 FOR 50MM x 50MM BOARDS WITH 4 NPTH"
- note added: "SQUARE WAVE GENERATOR"
- note removed: "4 WIRE KELVIN INPUT"
- note removed: "Banana plug socket holes ARE NOT not be the right size. Also need to be different colours"
- note removed: "CHECK THE FOLLOWING:- SWITCH = Fully Checked, diode fuse battery con"
- note removed: "DETERMINE IF THE COMPARATOR CAN SINK ENOUGH CURRENT DETERMINE IF A TRANSISTOR IS NEEDED ON THE OUTPUT, DETERMINE IF AC COUPLIG WILL REDUCE DC CURRENT DRAW"
- note removed: "NOT SETUP CORRECTLY YET MAY BE BETTER WITH 2 WIRE, OR LOOK AT TONE OHM SETUP"
- note removed: "REPLACE PART NUMBER WITH ONE FOR A 2.7V ZENER"
- note removed: "THIS ISNT RIGHT"
- note removed: "ZENER ISNT RIGHT"
- moved on the sheet: C1, C10, C2, C3, C4, C5, C6, C7, C8, C9, D1, D3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

Commit message: Minor updates
Minor Updates
Other:
- note added: "CHECK POST SIZE IS THE ONE DESIRED"
- note added: "Hirschmann black safety socket spade connector, 25A Red 972 355-101 Black 972 355-100 gold plated farnell £1.33 each"
- note removed: "BUZZER PART NEEDS CREATING FOR KMTG1203 AND FOOTPRINT NEEDS CORRECTING"
- note removed: "FIT EITHER Q1 OR R21"
- note removed: "NO CONNECT PINS IC, I.C._2, I.C._3"
Changed lines of the file:
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@@
 <sheet>
 <plain>
-<text x="119.38" y="-40.64" size="1.778" layer="91">NO CONNECT PINS IC, I.C._2, I.C._3</text>
 <text x="-190.5" y="-73.66" size="1.778" layer="91">REVERSE
 VOLTAGE
@@
 <text x="-185.42" y="-48.26" size="1.778" layer="91">ON/OFF</text>
 <text x="43.18" y="48.26" size="3.81" layer="91">WWW.GUVVY.CO.UK</text>
-<text x="261.62" y="-91.44" size="1.778" layer="91">FIT EITHER Q1 OR R21</text>
-<text x="358.14" y="-167.64" size="1.778" layer="91">BUZZER PART NEEDS CREATING FOR
- KMTG1203 AND FOOTPRINT NEEDS
-CORRECTING</text>
 <text x="325.12" y="-144.78" size="1.778" layer="91">DETERMINE IF THE COMPARATOR CAN
  SINK ENOUGH CURRENT DETERMINE
@@
 Fuse = checked
 Battery con = checked</text>
-<text x="-96.52" y="-147.32" size="1.778" layer="91">NEED HIGHER POWER INPUT RESISTORS FOR LARGE INPUT VOLTAGES</text>
+<text x="-88.9" y="-152.4" size="1.778" layer="91">NEED HIGHER POWER INPUT RESISTORS FOR LARGE INPUT VOLTAGES</text>
 <text x="-142.24" y="-83.82" size="1.778" layer="91">BD4827G-TR</text>
 <text x="243.84" y="-198.12" size="1.778" layer="91">SQUARE WAVE GENERATOR</text>
@@
 <text x="86.36" y="20.32" size="1.778" layer="91">FIDUCIALS</text>
 <text x="-261.62" y="-91.44" size="1.778" layer="91">DUAL FOOTPRINT. ONLY FIT ONE BATTERY HOLDER.</text>
+<text x="-88.9" y="-144.78" size="3.81" layer="91">CHECK POST SIZE IS THE ONE DESIRED</text>
+<text x="-81.28" y="-177.8" size="1.778" layer="91">Hirschmann black safety socket spade connector, 25A
+Red 972 355-101
+Black 972 355-100
+gold plated
+farnell £1.33 each </text>
 </plain>
 <instances>

Commit message: CAD A Release Version
CAD A Release Version
Moved battery inboard requiring moving of various components
Parts:
- renumbered U$1 to FID1, U$2 to FID2, U$3 to FID3, U$4 to FID4, VR3 to VR2
Other:
- note added: "MAY NEED HIGHER POWER INPUT RESISTORS FOR LARGE INPUT VOLTAGES"
- note removed: "NEED HIGHER POWER INPUT RESISTORS FOR LARGE INPUT VOLTAGES"
Changed lines of the file:
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@@
 <part name="SG1" library="KMTG1203" deviceset="BUZZER" device="BUZZER-KMTG1203"/>
 <part name="P+2" library="supply1" deviceset="VCC" device=""/>
-<part name="VR3" library="bourns" deviceset="3386-" device="F" value="1k"/>
+<part name="VR2" library="bourns" deviceset="3386-" device="F" value="1k"/>
 <part name="S1" library="SparkFun-Electromechanical" deviceset="SWITCH-SPDT" device="-SMD-A" value="C&amp;K COMPONENTS PCM12SMTR">
 <attribute name="MF" value="C&amp;K COMPONENTS"/>
@@
 <part name="TP2" library="TP_1MM_TH" deviceset="TP_1MM_TH" device="&quot;"/>
 <part name="TP4" library="TP_1MM_TH" deviceset="TP_1MM_TH" device="&quot;"/>
-<part name="U$1" library="adafruit" deviceset="FIDUCIAL" device=""/>
-<part name="U$2" library="adafruit" deviceset="FIDUCIAL" device=""/>
-<part name="U$3" library="adafruit" deviceset="FIDUCIAL" device=""/>
-<part name="U$4" library="adafruit" deviceset="FIDUCIAL" device=""/>
+<part name="FID1" library="adafruit" deviceset="FIDUCIAL" device=""/>
+<part name="FID2" library="adafruit" deviceset="FIDUCIAL" device=""/>
+<part name="FID3" library="adafruit" deviceset="FIDUCIAL" device=""/>
+<part name="FID4" library="adafruit" deviceset="FIDUCIAL" device=""/>
 <part name="SP4" library="buzzer" deviceset="KSS1201" device=""/>
 <part name="BAT1" library="SparkFun-Electromechanical" deviceset="BATTERY" device="FOB" value="CR2032"/>
@@
 Fuse = checked
 Battery con = checked</text>
-<text x="-88.9" y="-152.4" size="1.778" layer="91">NEED HIGHER POWER INPUT RESISTORS FOR LARGE INPUT VOLTAGES</text>
+<text x="-88.9" y="-152.4" size="1.778" layer="91">MAY NEED HIGHER POWER INPUT RESISTORS FOR LARGE INPUT VOLTAGES</text>
 <text x="-142.24" y="-83.82" size="1.778" layer="91">BD4827G-TR</text>
 <text x="243.84" y="-198.12" size="1.778" layer="91">SQUARE WAVE GENERATOR</text>
@@
 <instance part="SG1" gate="G$1" x="325.12" y="-165.1" rot="R270"/>
 <instance part="P+2" gate="VCC" x="48.26" y="-96.52"/>
-<instance part="VR3" gate="G$1" x="314.96" y="-139.7" rot="R180"/>
+<instance part="VR2" gate="G$1" x="314.96" y="-139.7" rot="R180"/>
 <instance part="S1" gate="1" x="-182.88" y="-55.88">
 <attribute name="MF" x="-182.88" y="-55.88" size="1.778" layer="96" display="off"/>
@@
 <instance part="TP2" gate="G$1" x="-119.38" y="-129.54" rot="R180"/>
 <instance part="TP4" gate="G$1" x="-93.98" y="-129.54"/>
-<instance part="U$1" gate="G$1" x="55.88" y="20.32"/>
-<instance part="U$2" gate="G$1" x="63.5" y="20.32"/>
-<instance part="U$3" gate="G$1" x="71.12" y="20.32"/>
-<instance part="U$4" gate="G$1" x="78.74" y="20.32"/>
+<instance part="FID1" gate="G$1" x="55.88" y="20.32"/>
+<instance part="FID2" gate="G$1" x="63.5" y="20.32"/>
+<instance part="FID3" gate="G$1" x="71.12" y="20.32"/>
+<instance part="FID4" gate="G$1" x="78.74" y="20.32"/>
 <instance part="SP4" gate="1" x="340.36" y="-167.64" rot="R270"/>
 <instance part="BAT1" gate="G$1" x="-243.84" y="-68.58" rot="R270"/>
@@
 <wire x1="314.96" y1="-144.78" x2="314.96" y2="-152.4" width="0.1524" layer="91"/>
 <pinref part="C14" gate="G$1" pin="1"/>
-<pinref part="VR3" gate="G$1" pin="3"/>
+<pinref part="VR2" gate="G$1" pin="3"/>
 </segment>
 </net>
@@
 <net name="VOUT_COMP" class="0">
 <segment>
-<pinref part="VR3" gate="G$1" pin="1"/>
+<pinref part="VR2" gate="G$1" pin="1"/>
 <wire x1="314.96" y1="-134.62" x2="314.96" y2="-132.08" width="0.1524" layer="91"/>
 <wire x1="314.96" y1="-132.08" x2="307.34" y2="-132.08" width="0.1524" layer="91"/>
@@
 <pinref part="U5" gate="A" pin="OUT"/>
 <junction x="284.48" y="-139.7"/>
-<pinref part="VR3" gate="G$1" pin="2"/>
+<pinref part="VR2" gate="G$1" pin="2"/>
 <wire x1="284.48" y1="-139.7" x2="281.94" y2="-139.7" width="0.1524" layer="91"/>
 <wire x1="307.34" y1="-139.7" x2="284.48" y2="-139.7" width="0.1524" layer="91"/>

Commit message: minor movement on the schematic
minor movement on the schematic
Parts:
- BAT1, C1, C6, C7, C9, D4, D6, FID1, FID2, FID3, FID4, LED1, LED2, LED3, PCB1, Q1, R1, R10, R11, R12, R13, R14, R15, R16, R17, R18, R19, R2, R20, R21, R3, R4, R5, R6, R7, R9, TP1, TP2, TP3, TP4, TP5, TP6, VR1, VR2: OC_FARNELL (none) -> unknown
- C10, C13: value 100nF -> 100n; MF (none) -> MULTICOMP; MPN (none) -> MC0402X104K100CT; OC_FARNELL (none) -> 1759380
- C11: value 10nF -> 10n; OC_FARNELL (none) -> unknown
- C12, C14, C2: value 10uF -> 10u; MF (none) -> MURATA; MPN (none) -> GRM188R61A106ME69D; OC_FARNELL (none) -> 2456110
- C3, C5, C8: MF (none) -> MULTICOMP; MPN (none) -> MC0402X104K100CT; OC_FARNELL (none) -> 1759380
- C4: value 470pF -> 470p; OC_FARNELL (none) -> unknown
- D2, D3, D5: MF (none) -> MULTICOMP; MPN (none) -> 1N4148W; OC_FARNELL (none) -> 1621821
- J3: value BNCPTH -> TE 5227161-1; MF (none) -> TE CONNECTIVITY / AMP; MPN (none) -> 5227161-1; OC_FARNELL (none) -> 1338762
- R8: value (none) -> 0.1R; OC_FARNELL (none) -> unknown
- S1: MF C&K COMPONENTS -> C & K COMPONENTS
- SG1: MF (none) -> KINGSTATE; MPN (none) -> KMTG1203; OC_FARNELL (none) -> 2215052
- SP4: value KSS1201 -> SPKR_PTH_6.5MM_PITCH
- U1: MF (none) -> ROHM; MPN (none) -> BD4827G-TR; OC_FARNELL (none) -> 2343050
- U2: MF (none) -> TEXAS INSTRUMENTS; OC_FARNELL (none) -> 2119784
- U3: MF (none) -> TEXAS INSTRUMENTS
- U4, U5: MF (none) -> MICROCHIP
Other:
- note added: "Needs adjustable resistance range. up to 200 ohm"
- moved on the sheet: C10, C13, C3, C5

Commit message: Updated part values and part number
Updated part values and part number
Parts:
- D4: value 2.7V -> 3.3V
- D6: value 2.7V -> DNF
- J1: value BANANA_CONN -> BANANA_CONN_BLACK; MF (none) -> CLIFF ELECTRONIC COMPONENTS; MPN (none) -> FCR14460; OC_FARNELL unknown -> 2392747
- J2: value BANANA_CONN -> BANANA_CONN_RED; MF (none) -> CLIFF ELECTRONIC COMPONENTS; MPN (none) -> FCR14461; OC_FARNELL unknown -> 2392748
- LED1: value (none) -> Red LED; MF (none) -> KINGBRIGHT; MPN (none) -> KP-1608SURCK; OC_FARNELL unknown -> 2290329
- LED2: value (none) -> Green LED; MF (none) -> KINGBRIGHT; MPN (none) -> KP-1608CGCK; OC_FARNELL unknown -> 2290328
- LED3: value (none) -> Yellow LED; MF (none) -> KINGBRIGHT; MPN (none) -> KP-1608SYCK; OC_FARNELL unknown -> 2290330
- Q1: MF (none) -> ON SEMICONDUCTOR; MPN (none) -> BC807-16LT1G; OC_FARNELL unknown -> 2317586
- R1, R13, R2: value 2k -> 2k 5%
- R10, R11: value (none) -> 100R 5%
- R12: value (none) -> 0R0
- R14: value (none) -> 2k 5%
- R15, R4: value 1M -> 1M 5%
- R16, R20: value 47k -> 47k 5%
- R17: value 100k -> 100k 5%
- R18, R21: value 1k -> 1k 5%
- R19: value 330R -> 330R 5%
- R3: value (none) -> 619R 0.1%; MF (none) -> TE CONNECTIVITY; MPN (none) -> CPF0402B619RE1; OC_FARNELL unknown -> 2330768
- R5: value (none) -> 1k 1%
- R6: value (none) -> 1k 0.1%; MF (none) -> WELWYN; MPN (none) -> PCF0402-R-1K-B-T1.; OC_FARNELL unknown -> 1108781
- R7: value (none) -> 150R 5%
- R8: value 0.1R -> 0.1R 1%; MF (none) -> PANASONIC ELECTRONIC COMPONENTS; MPN (none) -> ERJ3RSFR10V; OC_FARNELL unknown -> 1717759
- R9: value (none) -> 499k 1%; MF (none) -> PANASONIC ELECTRONIC COMPONENTS; MPN (none) -> ERJ3EKF4993V; OC_FARNELL unknown -> 2303291
- U2: MPN (none) -> TLV431BCDBZTG4; OC_FARNELL 2119784 -> 1053385
- VR1: value (none) -> 100k 10%; MF (none) -> BOURNS; MPN (none) -> 3386F-1-104TLF; OC_FARNELL unknown -> 9354581
- VR2: value 1k -> 1k 10%; MF (none) -> BOURNS; MPN (none) -> 3386F-1-102TLF; OC_FARNELL unknown -> 9354549
Other:
- note added: ""SICK OF BEIGE" DP5050 FOR 50MM x 50MM BOARDS WITH 4 NPTH"
- note added: "Alternatively: 8 x M3 screws n mm 4 x M3 standoffs n mm 4 x M3 standoffs n mm Laser cut or cnc acrylic sheets"
- note added: "CHECK POWER RATING"
- note added: "Determine which part fits. VISHAY M63M102KB30T607 1k potentiometer with knob Or BOURNS 3386F-1-102TLF"
- note added: "Hirschmann black safety socket spade connector, 25A Red 972 355-101 Black 972 355-100 gold plated farnell £1.33 each Cliff Electronic - FCR14460 - Black £0.72 chunky plastic with wire solder tab. Cliff Electronic - FCR14461- Red Right Angle Safety: Cliff Electronic FCR7350B - Black £2.11 (rapid) £4.27 farnell, CPC £1.96 Cliff Electronic FCR7350R - Red £2.11 (rapid) £4.27 farnell, CPC £1.96 Ali-Ex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"
- note added: "Precision 0.1% resistors appear to be more readily available in 0603 or 0805 rather than 0402 packages. and are cheapest in 0805 Change Rin, Rf and the Vref load resistor to 0.1% 0603 parts if cheaper or available"
- note added: "TH: 5mm pitch, 12.6mm dia farnell: 1823866 7.6mm pitch and 13.8mm dia farnell: 1022401 SMD 12x12mm Farnell: 1192551 PKLCS1212E4001-R1 12x12mm Farnell: 2443206 PKLCS1212E2400-R1 12.8x12.8mm Farnell: 2215053 round smd 2215050 PKLCS1212E2400-R1 PKMCS0909E4000-R1 mouser only KMTG1603 KMTG1203"
- note removed: "Hirschmann black safety socket spade connector, 25A Red 972 355-101 Black 972 355-100 gold plated farnell £1.33 each"
- note removed: "SICK OF BEIGE DP5050 FOR 50MM x 50MM BOARDS WITH 4 NPTH"
- moved on the sheet: C2, LED2, PCB1, R2, R20

Commit message: updated layout and parts
updated layout and parts
Parts:
- BAT1: value CR2032 -> DNF CR2032
- R18, R21: value 1k 5% -> 1k 1%
- U5: value Comparator -> MCP6541T-I/OT
Other:
- note added: "Change 499k to 0.1% , may need an 0603 or 0805 part. Change 0.1% 1k to a larger package so that it is not confused with the 1% 1k parts and is cheaper."
- note added: "NO LED DIRECTION INDICATOR ON PCB. NEEDS CORRECTING"
- note added: "THICKEN VCC LINE ON LAYOUT"
Changed lines of the file:
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@@
 <attribute name="OC_FARNELL" value="2317586"/>
 </part>
-<part name="R18" library="rcl" deviceset="R-EU_" device="R0402" value="1k 5%">
+<part name="R18" library="rcl" deviceset="R-EU_" device="R0402" value="1k 1%">
 <attribute name="MF" value=""/>
 <attribute name="MPN" value=""/>
@@
 <attribute name="OC_FARNELL" value="unknown"/>
 </part>
-<part name="R21" library="rcl" deviceset="R-EU_" device="R0402" value="1k 5%">
+<part name="R21" library="rcl" deviceset="R-EU_" device="R0402" value="1k 1%">
 <attribute name="MF" value=""/>
 <attribute name="MPN" value=""/>
@@
 </part>
 <part name="P+7" library="supply1" deviceset="VCC" device=""/>
-<part name="U5" library="MCP6541_SOT23-5" deviceset="MCP6541T-I/OT" device="" value="Comparator">
+<part name="U5" library="MCP6541_SOT23-5" deviceset="MCP6541T-I/OT" device="" value="MCP6541T-I/OT">
 <attribute name="MF" value="MICROCHIP"/>
 </part>
@@
 </part>
 <part name="SP4" library="buzzer" deviceset="KSS1201" device="" value="SPKR_PTH_6.5MM_PITCH"/>
-<part name="BAT1" library="SparkFun-Electromechanical" deviceset="BATTERY" device="FOB" value="CR2032">
+<part name="BAT1" library="SparkFun-Electromechanical" deviceset="BATTERY" device="FOB" value="DNF   CR2032">
 <attribute name="MF" value=""/>
 <attribute name="MPN" value=""/>
@@
 <text x="325.12" y="-124.46" size="1.778" layer="91">Determine which part fits. VISHAY M63M102KB30T607 1k potentiometer with knob
 Or BOURNS 3386F-1-102TLF</text>
+<text x="-121.92" y="-43.18" size="1.778" layer="91">NO LED DIRECTION INDICATOR ON PCB. NEEDS CORRECTING</text>
+<text x="-121.92" y="-27.94" size="1.778" layer="91">THICKEN VCC LINE ON LAYOUT</text>
+<text x="35.56" y="-162.56" size="1.778" layer="91">Change 499k to 0.1% , may need an 0603 or 0805 part.
+Change 0.1% 1k to a larger package so that it is not confused with the 1% 1k parts and is cheaper. </text>
 </plain>
 <instances>
@@
 <instance part="U5" gate="A" x="264.16" y="-142.24">
 <attribute name="MF" x="264.16" y="-142.24" size="1.778" layer="96" display="off"/>
+<attribute name="MPN" x="256.54" y="-162.56" size="1.778" layer="96" display="off"/>
 </instance>
 <instance part="SG1" gate="G$1" x="325.12" y="-165.1" rot="R270">

Commit message: minor updates
Other:
- note added: "MCP6001 Isc = +-23mA@5.5v, +-6mA@1.8V"
- note added: "MCP6541 Isc = +-30mA@5.5v, -2.5mA/+1.5mA@1.6V, ABS max +-30mA"
Changed lines of the file:
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@@
 <text x="35.56" y="-162.56" size="1.778" layer="91">Change 499k to 0.1% , may need an 0603 or 0805 part.
 Change 0.1% 1k to a larger package so that it is not confused with the 1% 1k parts and is cheaper. </text>
+<text x="165.1" y="-71.12" size="1.778" layer="91">MCP6001 Isc = +-23mA@5.5v, +-6mA@1.8V</text>
+<text x="256.54" y="-104.14" size="1.778" layer="91">MCP6541 Isc = +-30mA@5.5v, -2.5mA/+1.5mA@1.6V, ABS max +-30mA</text>
 </plain>
 <instances>
